File: gps_compass_circuit_atmega328/gps_compass.kicad_pcb (KiCad board)
At the start: 2 copper layers, 37 parts, among them SW1 SW_DIP_x05, U1 LSM303C, U2 MAX-M8C, U3 ATmega328P-A, U4 MCP1700x-330xxTT

Commit message: upd circuit
Parts:
- removed AE1: Antenna, Connector_Coaxial:U.FL_Hirose_U.FL-R-SMT-1_Vertical
- removed C_sup2: 3.9v200F, Capacitor_THT:C_Rect_L7.5mm_W6.5mm_P5.00mm
- removed Cd12, Cd13: 1uf, Capacitor_SMD:C_0603_1608Metric
- removed Cv1: 1uF, Capacitor_SMD:C_0603_1608Metric
- removed D2: BZV55B3V9, Diode_SMD:D_MiniMELF
- removed SW1: SW_DIP_x05, Library:SW_JS1300AQ
- removed U3: ATmega328P-A, Package_QFP:TQFP-32_7x7mm_P0.8mm
- removed U4: MCP1700x-330xxTT, Package_TO_SOT_SMD:SOT-23
- added C1: 0.1uF, Capacitor_SMD:C_0603_1608Metric, F.Cu at (180.7, 65.2)
- added C2: 22pF, Capacitor_SMD:C_0603_1608Metric, F.Cu at (172.7, 69.8)
- added C3: 22pF, Capacitor_SMD:C_0603_1608Metric, F.Cu at (172.7, 65.2)
- added C4: 22uF, Capacitor_SMD:C_0603_1608Metric, F.Cu at (193.4, 89.7)
- added Cgps1: 100pF, Capacitor_SMD:C_0603_1608Metric, F.Cu at (171.1, 88.7)
- added Cgps2: 100pF, Capacitor_SMD:C_0603_1608Metric, F.Cu at (175.1, 86.1)
- added Cgps3: 1uF, Capacitor_SMD:C_0603_1608Metric, F.Cu at (179.1, 86.1)
- added Cgps4: 100pF, Capacitor_SMD:C_0603_1608Metric, F.Cu at (179.1, 88.7)
- added JCompass1: Conn_01x05, Connector_PinSocket_2.54mm:PinSocket_1x05_P2.54mm_Vertical, F.Cu at (166.8, 87.2)
- added JGPS1: Conn_01x05, Connector_PinSocket_2.54mm:PinSocket_1x05_P2.54mm_Vertical, F.Cu at (162.2, 87.2)
- added L1: 4,7uH, Inductor_SMD:L_0603_1608Metric, F.Cu at (194.0, 87.2)
- added Led1: LED, LED_THT:LED_D3.0mm, F.Cu at (147.0, 87.7)
- added Lgps1: 33nH, Inductor_SMD:L_0603_1608Metric, F.Cu at (171.1, 86.1)
- added Lgps2: 33nH, Inductor_SMD:L_0603_1608Metric, F.Cu at (171.1, 93.7)
- added R1: 1M, Capacitor_SMD:C_0603_1608Metric, F.Cu at (176.7, 65.2)
- added R2: 100K, Capacitor_SMD:C_0603_1608Metric, F.Cu at (176.7, 67.7)
- added Rgps1: 200R, Resistor_SMD:R_0603_1608Metric, F.Cu at (171.1, 91.2)
- added Rgps2: 200R, Resistor_SMD:R_0603_1608Metric, F.Cu at (171.1, 96.2)
- added Rled1: 700R, Resistor_SMD:R_0603_1608Metric, F.Cu at (153.3, 86.1)
- added SWLed1: SW_Reset, Button_Switch_THT:SW_PUSH_6mm, F.Cu at (125.2, 95.9)
- added SW_MCU1: SW_DPDT_x2, Connector_PinSocket_2.54mm:PinSocket_1x03_P2.54mm_Vertical, F.Cu at (200.4, 77.0)
- added Y1: Crystal, Crystal:Resonator-2Pin_W10.0mm_H5.0mm, F.Cu at (174.2, 60.4)
- C_sup1: value 3.9v200F -> 2.7v200F; footprint Capacitor_THT:C_Rect_L7.5mm_W6.5mm_P5.00mm -> Capacitor_THT:C_Rect_L9.0mm_W2.5mm_P7.50mm_MKT
- SWReset1: footprint Button_Switch_SMD:SW_SPST_Omron_B3FS-101xP -> Button_Switch_THT:SW_PUSH_6mm
- SW_main_switch1: footprint Connector_PinHeader_2.54mm:PinHeader_1x03_P2.54mm_Vertical -> Connector_PinSocket_2.54mm:PinSocket_1x03_P2.54mm_Vertical
- U1: value LSM303C -> ATmega328P-A; footprint Package_LGA:LGA-12_2x2mm_P0.5mm -> Package_QFP:TQFP-32_7x7mm_P0.8mm
- U2: value MAX-M8C -> TPS613221ADBV; footprint RF_GPS:ublox_MAX -> Package_TO_SOT_SMD:SOT-23-5
- moved Cd10 95.4 mm to (151.4, 91.7)
- moved Cd2 86.8 mm to (147.4, 91.7)
- moved Cd6 83.1 mm to (143.8, 97.6)
- moved Cd7 83.1 mm to (139.8, 97.6)
- moved Cd9 79.1 mm to (143.8, 95.1)
- moved Cd8 79.1 mm to (135.8, 102.6)
- moved Cd5 79.1 mm to (135.8, 95.1)
- moved JDisplay1 75.6 mm to (134.3, 88.4)
- moved Cd4 75.1 mm to (135.8, 100.1)
- moved Cd11 75.1 mm to (139.8, 95.1)
- moved Cd3 75.1 mm to (139.8, 100.1)
- moved Cd1 67.1 mm to (135.8, 97.6)
- moved D1 58.6 mm to (199.5, 86.1), turned to 0 degrees
- moved SC_1 54.4 mm to (205.0, 77.0)
- moved SW_main_switch1 53.6 mm to (189.8, 81.1)
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Connections:
- SC_1 pad 2: Net-(SC_1-Pad2) -> GND
- SC_2 pad 1: Net-(SC_1-Pad2) -> Net-(R_cells1-Pad2)
- SW_main_switch1 pad 3: Net-(SW_main_switch1-Pad3) -> Power_level
- U1 pad 1: SCL -> gps_rx
- U1 pad 10: +3V3 -> Display_CS
- U1 pad 12: unconnected-(U1-Pad12) -> B1
- U1 pad 2: unconnected-(U1-Pad2) -> Display_DA
- U1 pad 3: unconnected-(U1-Pad3) -> GND
- U1 pad 4: SDA -> +3V3
- U1 pad 5: unconnected-(U1-Pad5) -> GND
- U1 pad 6: GND -> +3V3
- U1 pad 7: unconnected-(U1-Pad7) -> Net-(C2-Pad1)
- U1 pad 8: GND -> Net-(C3-Pad1)
- U1 pad 9: +3V3 -> Display_WR
- U2 pad 1: GND -> Net-(L1-Pad2)
- U2 pad 2: gps_tx -> GND
- U2 pad 3: gps_rx -> unconnected-(U2-Pad3)
- U2 pad 4: unconnected-(U2-Pad4) -> VCC
