File: gps_compass_circuit_atmega328/gps_compass_display.kicad_sch (KiCad schematic)
At the start: 12 parts

Commit message: upd circuit
Parts:
- added Led1: LED, LED_THT:LED_D3.0mm, symbol Device:LED
- added Rled1: 700R, Resistor_SMD:R_0603_1608Metric, symbol pspice:R
- added SWLed1: SW_Reset, Button_Switch_THT:SW_PUSH_6mm, symbol Switch:SW_DIP_x01
Connections:
- net +3V3: now also Rled1.2
- net GND: now also SWLed1.1
- new net: Led1.1 (K), SWLed1.2
- new net: Led1.2 (A), Rled1.1
Changed lines of the file:
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@@
+    (stroke (width 0) (type default) (color 0 0 0 0))
+  )
+  (wire (pts (xy 66.04 121.92) (xy 66.04 127))
     (stroke (width 0) (type default) (color 0 0 0 0))
   )
@@
     (stroke (width 0) (type default) (color 0 0 0 0))
   )
+  (wire (pts (xy 66.04 105.41) (xy 66.04 109.22))
+    (stroke (width 0) (type default) (color 0 0 0 0))
+  )
   (wire (pts (xy 146.05 129.54) (xy 146.05 132.08))
     (stroke (width 0) (type default) (color 0 0 0 0))
@@
     (stroke (width 0) (type default) (color 0 0 0 0))
   )
+  (wire (pts (xy 66.04 93.98) (xy 66.04 97.79))
+    (stroke (width 0) (type default) (color 0 0 0 0))
+  )
   (wire (pts (xy 162.56 96.52) (xy 137.16 96.52))
     (stroke (width 0) (type default) (color 0 0 0 0))
@@
   )
   (wire (pts (xy 140.97 81.28) (xy 162.56 81.28))
+    (stroke (width 0) (type default) (color 0 0 0 0))
+  )
+  (wire (pts (xy 66.04 72.39) (xy 66.04 78.74))
     (stroke (width 0) (type default) (color 0 0 0 0))
   )
@@
     )
   )
+  (symbol (lib_id "power:GND") (at 66.04 72.39 180) (unit 1)
+    (in_bom yes) (on_board yes) (fields_autoplaced)
+    (property "Reference" "#PWR0102" (id 0) (at 66.04 66.04 0)
+      (effects (font (size 1.27 1.27)) hide)
+    )
+    (property "Value" "GND" (id 1) (at 66.0401 68.58 90)
+      (effects (font (size 1.27 1.27)) (justify right))
+    )
+    (property "Footprint" "" (id 2) (at 66.04 72.39 0)
+      (effects (font (size 1.27 1.27)) hide)
+    )
+    (property "Datasheet" "" (id 3) (at 66.04 72.39 0)
+      (effects (font (size 1.27 1.27)) hide)
+    )
+    (pin "1")
+  )
   (symbol (lib_id "Device:C") (at 125.73 121.92 90) (unit 1)
     (in_bom yes) (on_board yes)
@@
     (pin "2")
   )
+  (symbol (lib_id "Device:LED") (at 66.04 101.6 270) (unit 1)
+    (in_bom yes) (on_board yes) (fields_autoplaced)
+    (property "Reference" "Led1" (id 0) (at 72.39 100.0125 0))
+    (property "Value" "LED" (id 1) (at 69.85 100.0125 0))
+    (property "Footprint" "LED_THT:LED_D3.0mm" (id 2) (at 66.04 101.6 0)
+      (effects (font (size 1.27 1.27)) hide)
+    )
+    (property "Datasheet" "~" (id 3) (at 66.04 101.6 0)
+      (effects (font (size 1.27 1.27)) hide)
+    )
+    (pin "1")
+    (pin "2")
+  )
   (symbol (lib_id "Device:C") (at 146.05 114.3 90) (unit 1)
     (in_bom yes) (on_board yes)
@@
     (pin "1")
     (pin "2")
+  )
+  (symbol (lib_id "pspice:R") (at 66.04 115.57 0) (unit 1)
+    (in_bom yes) (on_board yes) (fields_autoplaced)
+    (property "Reference" "Rled1" (id 0) (at 72.39 115.57 90))
+    (property "Value" "700R" (id 1) (at 69.85 115.57 90))
+    (property "Footprint" "Resistor_SMD:R_0603_1608Metric" (id 2) (at 66.04 115.57 0)
+      (effects (font (size 1.27 1.27)) hide)
+    )
+    (property "Datasheet" "~" (id 3) (at 66.04 115.57 0)
+      (effects (font (size 1.27 1.27)) hide)
+    )
+    (pin "1")
+    (pin "2")
+  )
+  (symbol (lib_id "power:+3V3") (at 66.04 127 180) (unit 1)
+    (in_bom yes) (on_board yes) (fields_autoplaced)
+    (property "Reference" "#PWR0101" (id 0) (at 66.04 123.19 0)
+      (effects (font (size 1.27 1.27)) hide)
+    )
+    (property "Value" "+3V3" (id 1) (at 66.0401 130.81 90)
+      (effects (font (size 1.27 1.27)) (justify left))
+    )
+    (property "Footprint" "" (id 2) (at 66.04 127 0)
+      (effects (font (size 1.27 1.27)) hide)
+    )
+    (property "Datasheet" "" (id 3) (at 66.04 127 0)
+      (effects (font (size 1.27 1.27)) hide)
+    )
+    (pin "1")
   )
   (symbol (lib_id "Device:C") (at 134.62 101.6 90) (unit 1)
@@
     (pin "1")
   )
+  (symbol (lib_id "Switch:SW_DIP_x01") (at 66.04 86.36 270) (unit 1)
+    (in_bom yes) (on_board yes) (fields_autoplaced)
+    (property "Reference" "SWLed1" (id 0) (at 71.12 86.36 0))
+    (property "Value" "SW_Reset" (id 1) (at 71.12 86.36 0)
+      (effects (font (size 1.27 1.27)) hide)
+    )
+    (property "Footprint" "Button_Switch_THT:SW_PUSH_6mm" (id 2) (at 66.04 86.36 0)
+      (effects (font (size 1.27 1.27)) hide)
+    )
+    (property "Datasheet" "~" (id 3) (at 66.04 86.36 0)
+      (effects (font (size 1.27 1.27)) hide)
+    )
+    (pin "1")
+    (pin "2")
+  )
   (symbol (lib_id "power:GND") (at 127 105.41 0) (unit 1)
