File: gps_compass_circuit_atmega328_7seg_battery/gps_compass.kicad_pcb (KiCad board)
At the start: 2 copper layers, 80 x 46 mm, 31 parts, among them J1 USB_C_Receptacle_PowerOnly_6P, J2 Micro_SD_Card, Q1 MMBTA92, U2 ESP32-WROOM-32U, U3 LTC4054ES5-4.2

Commit message: Aggiornato con circuito incompleto
Parts:
- added C5: 1uF, Capacitor_SMD:C_0805_2012Metric_Pad1.18x1.45mm_HandSolder, B.Cu at (124.4, 61.6)
- added C6: 0,1uF, Capacitor_SMD:C_0805_2012Metric_Pad1.18x1.45mm_HandSolder, B.Cu at (133.3, 63.9)
- added C7: 220uF, Capacitor_SMD:C_1206_3216Metric_Pad1.33x1.80mm_HandSolder, B.Cu at (133.8, 69.2)
- added C8: 220uF, Capacitor_SMD:C_1206_3216Metric_Pad1.33x1.80mm_HandSolder, B.Cu at (133.8, 66.4)
- added LED1: LED, LED_THT:LED_D3.0mm, F.Cu at (114.0, 44.1)
- added R6: R, Resistor_SMD:R_0603_1608Metric_Pad0.98x0.95mm_HandSolder, B.Cu at (124.4, 58.1)
- added U1: MCP1700x-330xxTT, Package_TO_SOT_SMD:SOT-23, B.Cu at (128.6, 64.8)
- C3, C4, L1, SWen1, SWprog1: moved to F.Cu
- GY-271: renamed from Jgy-271; footprint mia_libreria:BMP280 -> mia_libreria:GY-271
- Oled1: renamed from JOled1; value Conn_01x04_Shielded -> display_oled
- lcd1: renamed from Jlcd1; value Conn_01x05_Shielded -> display_lcd
- moved ESP32 144.5 mm to (164.7, 73.8), turned to -170 degrees
- moved SWprog1 142.7 mm to (113.7, 64.0), turned to -90 degrees
- moved C1 137.8 mm to (128.5, 61.6), turned to 0 degrees
- moved SWen1 136.6 mm to (117.8, 64.0), turned to 90 degrees
- moved microsd1 131.2 mm to (148.1, 66.8)
- moved R5 130.6 mm to (124.4, 56.4)
- moved C2 127.0 mm to (122.6, 65.9), turned to 0 degrees
- moved Q1 122.7 mm to (128.6, 69.0)
- moved Serial1 121.6 mm to (154.8, 33.3), turned to -90 degrees
- moved U2 120.5 mm to (139.4, 42.0), turned to -90 degrees
- moved R3 119.0 mm to (124.6, 63.7)
- moved J1 118.1 mm to (114.3, 56.5), turned to 90 degrees
- moved BT1 114.2 mm to (118.7, 56.4), turned to -90 degrees
- moved MAIN1 112.4 mm to (131.6, 74.5)
- moved U3 110.7 mm to (123.3, 69.0), turned to 0 degrees
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- renumbered SWesp32 to ESP32, SWgps1 to MAIN1, JSerial1 to Serial1, J2 to microsd1
Connections:
- MAIN1 pad 2: Net-(BT1-+) -> Net-(MAIN1-B)
- Serial1 pad 1: Net-(JSerial1-Pin_1) -> GND
- Serial1 pad 3: GND -> Net-(Serial1-Pin_3)
- U2 pad 35: Net-(JSerial1-Pin_1) -> Net-(Serial1-Pin_3)
- U2 pad 8: unconnected-(U2-IO32-Pad8) -> Net-(LED1-A)
Routing:
- net B6: track 0.00 -> 50.3 mm
- net SDA: track 0.00 -> 49.4 mm
- net Net-(SWen1-B): track 0.00 -> 45.4 mm, vias 0 -> 1
- net B5: track 0.00 -> 44.9 mm
- net VCC: track 0.00 -> 44.7 mm, vias 0 -> 2
- net +3V3: track 0.00 -> 43.5 mm
- net Net-(SWprog1-A): track 0.00 -> 41.7 mm, vias 0 -> 1
- net MOSI: track 0.00 -> 41.4 mm
- net Net-(Serial1-Pin_3): track 0.00 -> 39.7 mm, vias 0 -> 1
- net SCL: track 0.00 -> 39.2 mm
- net Net-(ESP32-B): track 0.00 -> 37.4 mm, vias 0 -> 1
- net Net-(Serial1-Pin_2): track 0.00 -> 35.3 mm, vias 0 -> 1
- net CLK: track 0.00 -> 34.7 mm
- net Net-(LED1-A): track 0.00 -> 33.9 mm
- net MISO: track 0.00 -> 33.2 mm
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- added copper zone on B.Cu, net GND
- added copper zone on F.Cu, net GND
Other:
- outline, holes or cut-outs redrawn
