File: gps_compass_circuit_atmega328_7seg_battery/gps_compass.kicad_sch (KiCad schematic)
At the start: 37 parts, among them J1 USB_C_Receptacle_PowerOnly_6P, J2 Micro_SD_Card, Q1 MMBTA92, U1 MCP1700x-330xxTT, U2 ESP32-WROOM-32U, U3 LTC4054ES5-4.2

Commit message: Aggiornato con circuito incompleto
Parts:
- added C8: 220uF, Capacitor_SMD:C_1206_3216Metric_Pad1.33x1.80mm_HandSolder, symbol Device:C
- C7: value 100uF -> 220uF; footprint Capacitor_SMD:C_0805_2012Metric_Pad1.18x1.45mm_HandSolder -> Capacitor_SMD:C_1206_3216Metric_Pad1.33x1.80mm_HandSolder
- GY-271: renamed from Jgy-271; footprint mia_libreria:BMP280 -> mia_libreria:GY-271
- renumbered SWesp32 to ESP32, D1 to LED1, SWgps1 to MAIN1, JOled1 to Oled1, JSerial1 to Serial1, Jlcd1 to lcd1, J2 to microsd1
Connections:
- net GND: now also Serial1.1 (Pin_1), C8.2; no longer Serial1.3 (Pin_3), Serial1.SH (Shield)
- net at C6.1, C7.1, MAIN1.2 (B)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: now also C8.1
- net at U2.35 (TXD0/IO1): now also Serial1.3 (Pin_3); no longer Serial1.1 (Pin_1)
- no-connect marks 23 -> 26
Other:
- moved on the sheet: C6, C7, MAIN1, Serial1
