File: gps_compass_circuit_atmega328_7seg/gps_compass.kicad_pcb (KiCad board)
At the start: 2 copper layers, 40 parts, among them U1 LSM303C, U3 ATmega328P-A, U4 MCP1700x-330xxTT, Y1 Crystal

Commit message: Aggiornato circuito
Parts:
- removed C_sup2: 3.9v200F, Capacitor_THT:C_Rect_L9.0mm_W2.5mm_P7.50mm_MKT
- removed U1: LSM303C, Package_LGA:LGA-12_2x2mm_P0.5mm
- added J1: Conn_01x05, Connector_PinSocket_2.54mm:PinSocket_1x05_P2.54mm_Vertical, F.Cu at (221.8, 60.9)
- JGPS1: value Conn_01x06 -> Conn_01x05; footprint Connector_PinSocket_2.54mm:PinSocket_1x06_P2.54mm_Vertical -> Connector_PinSocket_2.54mm:PinSocket_1x05_P2.54mm_Vertical
- SWLed1, SWReset1: footprint Button_Switch_SMD:SW_SPST_Omron_B3FS-101xP -> Button_Switch_THT:SW_PUSH_6mm
- moved D1 83.0 mm to (202.4, 60.3)
- moved SW_main_switch1 80.8 mm to (197.2, 60.9)
- moved Lgps1 79.7 mm to (234.1, 62.3)
- moved Rsda1 75.8 mm to (234.1, 59.8)
- moved Rled1 75.4 mm to (255.0, 58.2)
- moved Cgps4 74.7 mm to (230.1, 62.3)
- moved Cgps2 70.7 mm to (230.1, 59.8)
- moved Rscl1 70.7 mm to (226.1, 59.8)
- moved Cgps3 70.3 mm to (230.1, 64.9)
- moved Rgps1 69.9 mm to (226.1, 69.9)
- moved U4 68.6 mm to (201.9, 64.2)
- moved JDisplay1 68.6 mm to (244.8, 50.7)
- moved Led1 68.4 mm to (248.8, 59.7)
- moved C1 68.2 mm to (237.4, 41.4)
- moved C2 68.2 mm to (233.4, 43.5)
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Connections:
- JGPS1 pad 1: unconnected-(JGPS1-Pad1) -> Net-(Rgps1-Pad2)
- JGPS1 pad 2: Net-(Rgps1-Pad2) -> Net-(Rgps2-Pad2)
- JGPS1 pad 3: Net-(Rgps2-Pad2) -> Net-(Cgps3-Pad1)
- JGPS1 pad 4: Net-(Cgps3-Pad1) -> Net-(Cgps3-Pad2)
- JGPS1 pad 5: Net-(Cgps3-Pad2) -> unconnected-(JGPS1-Pad5)

Commit message: upt circuit
Parts:
- removed J1: Conn_01x05, Connector_PinSocket_2.54mm:PinSocket_1x05_P2.54mm_Vertical
- added JCompass1: Conn_01x05, Connector_PinSocket_2.54mm:PinSocket_1x05_P2.54mm_Vertical, F.Cu at (222.8, 57.3)
- moved C_sup1 3.74 mm to (186.5, 61.2)
- moved Cgps3 3.74 mm to (231.1, 61.2)
- moved Cv1 3.74 mm to (195.5, 73.1)
- moved Lgps2 3.74 mm to (227.1, 61.2)
- moved Rgps1 3.74 mm to (227.1, 66.3)
- moved SC_2 3.74 mm to (196.4, 67.0)
- moved Y1 3.74 mm to (235.9, 30.5)
- moved C1 3.74 mm to (238.4, 37.8)
- moved C2 3.74 mm to (234.3, 39.9)
- moved C3 3.74 mm to (242.4, 35.3)
- moved Cdtr1 3.74 mm to (217.0, 40.6)
- moved Cgps1 3.74 mm to (227.1, 58.7)
- moved Cgps2 3.74 mm to (231.1, 56.2)
- moved Cgps4 3.74 mm to (231.1, 58.7)
- moved D1 3.74 mm to (203.4, 56.6)
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
Commit message: Aggiornamenti vari
Parts:
- removed SJoystick1: JS1300AQ, Library:SW_JS1300AQ
- added SW1: SW_SPST, Button_Switch_THT:SW_PUSH_6mm, F.Cu at (23.2, 24.6)
- added SW2: SW_SPST, Button_Switch_THT:SW_PUSH_6mm, F.Cu at (23.2, 33.2)
- added SW3: SW_SPST, Button_Switch_THT:SW_PUSH_6mm, F.Cu at (23.2, 41.7)
- added SW4: SW_SPST, Button_Switch_THT:SW_PUSH_6mm, F.Cu at (23.2, 50.3)
- added SW5: SW_SPST, Button_Switch_THT:SW_PUSH_6mm, F.Cu at (23.2, 58.8)
- added SW6: SW_SPST, Button_Switch_THT:SW_PUSH_6mm, F.Cu at (23.2, 67.4)
- JCompass1: value Conn_01x05 -> GY-271; footprint Connector_PinSocket_2.54mm:PinSocket_1x05_P2.54mm_Vertical -> mia_libreria:GY-271
- JDisplay1: footprint Connector_PinSocket_2.54mm:PinSocket_1x05_P2.54mm_Vertical -> mia_libreria:display_7_segm_4_digits
- SC_1, SC_2: footprint Connector_PinSocket_2.54mm:PinSocket_1x02_P2.54mm_Vertical -> mia_libreria:solar_panel
- moved U3 228.5 mm to (31.1, 97.3)
- moved C3 226.0 mm to (23.2, 90.7)
- moved R1 222.8 mm to (23.2, 93.2)
- moved C1 220.4 mm to (23.2, 85.7)
- moved R2 219.6 mm to (23.2, 95.8)
- moved C2 216.6 mm to (23.2, 88.2)
- moved Y1 201.5 mm to (40.0, 78.0)
- moved JDisplay1 195.2 mm to (52.9, 76.6)
- moved Cdtr1 184.0 mm to (33.8, 57.2)
- moved SWReset1 179.7 mm to (23.2, 75.9)
- moved Led1 176.0 mm to (75.0, 77.8)
- moved Rled1 176.0 mm to (81.3, 76.3)
- moved SWLed1 176.0 mm to (75.4, 68.5)
- moved JMicroSD1 167.0 mm to (40.1, 47.9)
- moved Rreset1 153.8 mm to (33.8, 59.7)
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Connections:
- U3 pad 11: unconnected-(U3-Pad11) -> B6
