File: gps_compass_circuit_atmega328_7seg/gps_compass_GPS.kicad_sch (KiCad schematic)
At the start: 12 parts, among them U1 LSM303C

Commit message: Aggiornato circuito
Parts:
- removed JGPS1: Conn_01x06, Connector_PinSocket_2.54mm:PinSocket_1x06_P2.54mm_Vertical, symbol Connector_Generic:Conn_01x06
- removed U1: LSM303C, Package_LGA:LGA-12_2x2mm_P0.5mm, symbol Sensor_Motion:LSM303C
- added J1, JGPS1: Conn_01x05, Connector_PinSocket_2.54mm:PinSocket_1x05_P2.54mm_Vertical, symbol Connector_Generic:Conn_01x05
Connections:
- net +3V3: now also J1.1 (Pin_1)
- net GND: now also J1.2 (Pin_2)
- net SCL: now also J1.3 (Pin_3)
- net SDA: now also J1.4 (Pin_4)
- net at Cgps3.2, Cgps4.2, Lgps2.2: now also JGPS1.4 (Pin_4)
- net at Cgps3.1, Cgps4.1, Lgps1.2: now also JGPS1.3 (Pin_3)
- net at Rgps2.2: now also JGPS1.2 (Pin_2)
- net at Rgps1.2: now also JGPS1.1 (Pin_1)
- no-connect marks 6 -> 2
Other:
- moved on the sheet: Rscl1, Rsda1

Commit message: upt circuit
Parts:
- renumbered J1 to JCompass1
Other:
- moved on the sheet: Cgps3, Cgps4
Changed lines of the file:
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@@
 (kicad_sch (version 20211123) (generator eeschema)
   (paper "A4")
-  (junction (at 180.34 68.58) (diameter 0) (color 0 0 0 0)
-  )
-  (junction (at 180.34 60.96) (diameter 0) (color 0 0 0 0)
+  (junction (at 184.15 68.58) (diameter 0) (color 0 0 0 0)
+  )
+  (junction (at 184.15 60.96) (diameter 0) (color 0 0 0 0)
   )
   (junction (at 60.96 82.55) (diameter 0) (color 0 0 0 0)
@@
   (junction (at 163.83 85.09) (diameter 0) (color 0 0 0 0)
   )
-  (junction (at 172.72 60.96) (diameter 0) (color 0 0 0 0)
+  (junction (at 176.53 60.96) (diameter 0) (color 0 0 0 0)
   )
   (junction (at 71.12 80.01) (diameter 0) (color 0 0 0 0)
@@
   (junction (at 60.96 62.23) (diameter 0) (color 0 0 0 0)
   )
-  (junction (at 172.72 68.58) (diameter 0) (color 0 0 0 0)
+  (junction (at 176.53 68.58) (diameter 0) (color 0 0 0 0)
   )
   (no_connect (at 86.36 85.09))
@@
     (stroke (width 0) (type default) (color 0 0 0 0))
   )
-  (wire (pts (xy 158.75 85.09) (xy 163.83 85.09))
+  (wire (pts (xy 156.21 85.09) (xy 163.83 85.09))
     (stroke (width 0) (type default) (color 0 0 0 0))
   )
@@
     (stroke (width 0) (type default) (color 0 0 0 0))
   )
-  (wire (pts (xy 158.75 87.63) (xy 170.18 87.63))
+  (wire (pts (xy 156.21 87.63) (xy 170.18 87.63))
     (stroke (width 0) (type default) (color 0 0 0 0))
   )
@@
     (stroke (width 0) (type default) (color 0 0 0 0))
   )
-  (wire (pts (xy 200.66 60.96) (xy 180.34 60.96))
+  (wire (pts (xy 200.66 60.96) (xy 184.15 60.96))
     (stroke (width 0) (type default) (color 0 0 0 0))
   )
@@
     (stroke (width 0) (type default) (color 0 0 0 0))
   )
-  (wire (pts (xy 167.64 68.58) (xy 172.72 68.58))
+  (wire (pts (xy 167.64 68.58) (xy 176.53 68.58))
     (stroke (width 0) (type default) (color 0 0 0 0))
   )
@@
     (stroke (width 0) (type default) (color 0 0 0 0))
   )
-  (wire (pts (xy 172.72 68.58) (xy 180.34 68.58))
-    (stroke (width 0) (type default) (color 0 0 0 0))
-  )
-  (wire (pts (xy 180.34 68.58) (xy 198.12 68.58))
+  (wire (pts (xy 176.53 68.58) (xy 184.15 68.58))
+    (stroke (width 0) (type default) (color 0 0 0 0))
+  )
+  (wire (pts (xy 184.15 68.58) (xy 198.12 68.58))
     (stroke (width 0) (type default) (color 0 0 0 0))
   )
@@
     (stroke (width 0) (type default) (color 0 0 0 0))
   )
-  (wire (pts (xy 172.72 60.96) (xy 167.64 60.96))
+  (wire (pts (xy 176.53 60.96) (xy 167.64 60.96))
     (stroke (width 0) (type default) (color 0 0 0 0))
   )
@@
     (stroke (width 0) (type default) (color 0 0 0 0))
   )
-  (wire (pts (xy 180.34 60.96) (xy 172.72 60.96))
-    (stroke (width 0) (type default) (color 0 0 0 0))
-  )
-  (global_label "gps_rx" (shape input) (at 158.75 87.63 180) (fields_autoplaced)
+  (wire (pts (xy 184.15 60.96) (xy 176.53 60.96))
+    (stroke (width 0) (type default) (color 0 0 0 0))
+  )
+  (global_label "gps_rx" (shape input) (at 156.21 87.63 180) (fields_autoplaced)
     (effects (font (size 1.27 1.27)) (justify right))
-    (property "Riferimenti inter-foglio" "${INTERSHEET_REFS}" (id 0) (at 150.2288 87.5506 0)
+    (property "Riferimenti inter-foglio" "${INTERSHEET_REFS}" (id 0) (at 147.6888 87.5506 0)
       (effects (font (size 1.27 1.27)) (justify right) hide)
     )
   )
-  (global_label "gps_tx" (shape output) (at 158.75 85.09 180) (fields_autoplaced)
+  (global_label "gps_tx" (shape output) (at 156.21 85.09 180) (fields_autoplaced)
     (effects (font (size 1.27 1.27)) (justify right))
-    (property "Riferimenti inter-foglio" "${INTERSHEET_REFS}" (id 0) (at 150.2893 85.0106 0)
+    (property "Riferimenti inter-foglio" "${INTERSHEET_REFS}" (id 0) (at 147.7493 85.0106 0)
       (effects (font (size 1.27 1.27)) (justify right) hide)
     )
@@
   )
   (symbol (lib_id "Device:C") (at 170.18 93.98 0) (unit 1)
-    (in_bom yes) (on_board yes) (fields_autoplaced)
-    (property "Reference" "Cgps2" (id 0) (at 173.99 92.7099 0)
-      (effects (font (size 1.27 1.27)) (justify left))
-    )
-    (property "Value" "100pF" (id 1) (at 173.99 95.2499 0)
+    (in_bom yes) (on_board yes)
+    (property "Reference" "Cgps2" (id 0) (at 172.72 92.71 0)
+      (effects (font (size 1.27 1.27)) (justify left))
+    )
+    (property "Value" "100pF" (id 1) (at 172.72 95.25 0)
       (effects (font (size 1.27 1.27)) (justify left))
     )
@@
   (symbol (lib_id "Device:C") (at 163.83 93.98 0) (unit 1)
     (in_bom yes) (on_board yes)
-    (property "Reference" "Cgps1" (id 0) (at 156.21 92.71 0)
-      (effects (font (size 1.27 1.27)) (justify left))
-    )
-    (property "Value" "100pF" (id 1) (at 156.21 95.25 0)
+    (property "Reference" "Cgps1" (id 0) (at 154.94 92.71 0)
+      (effects (font (size 1.27 1.27)) (justify left))
+    )
+    (property "Value" "100pF" (id 1) (at 154.94 95.25 0)
       (effects (font (size 1.27 1.27)) (justify left))
     )
@@
   )
   (symbol (lib_id "pspice:INDUCTOR") (at 161.29 68.58 0) (unit 1)
-    (in_bom yes) (on_board yes) (fields_autoplaced)
-    (property "Reference" "Lgps2" (id 0) (at 161.29 62.23 0))
-    (property "Value" "33nH" (id 1) (at 161.29 64.77 0))
+    (in_bom yes) (on_board yes)
+    (property "Reference" "Lgps2" (id 0) (at 161.29 69.85 0))
+    (property "Value" "33nH" (id 1) (at 161.29 72.39 0))
     (property "Footprint" "Inductor_SMD:L_0603_1608Metric" (id 2) (at 161.29 68.58 0)
       (effects (font (size 1.27 1.27)) hide)
@@
     (pin "2")
   )
-  (symbol (lib_id "Device:C") (at 180.34 64.77 0) (unit 1)
-    (in_bom yes) (on_board yes)
-    (property "Reference" "Cgps4" (id 0) (at 177.8 62.23 0)
-      (effects (font (size 1.27 1.27)) (justify left))
-    )
-    (property "Value" "100pF" (id 1) (at 180.34 67.31 0)
-      (effects (font (size 1.27 1.27)) (justify left))
-    )
-    (property "Footprint" "Capacitor_SMD:C_0603_1608Metric" (id 2) (at 181.3052 68.58 0)
-      (effects (font (size 1.27 1.27)) hide)
-    )
-    (property "Datasheet" "~" (id 3) (at 180.34 64.77 0)
-      (effects (font (size 1.27 1.27)) hide)
-    )
-    (pin "1")
-    (pin "2")
-  )
-  (symbol (lib_id "Device:C") (at 172.72 64.77 0) (unit 1)
-    (in_bom yes) (on_board yes)
-    (property "Reference" "Cgps3" (id 0) (at 170.18 62.23 0)
-      (effects (font (size 1.27 1.27)) (justify left))
-    )
-    (property "Value" "1uF" (id 1) (at 172.72 67.31 0)
-      (effects (font (size 1.27 1.27)) (justify left))
-    )
-    (property "Footprint" "Capacitor_SMD:C_0603_1608Metric" (id 2) (at 173.6852 68.58 0)
-      (effects (font (size 1.27 1.27)) hide)
-    )
-    (property "Datasheet" "~" (id 3) (at 172.72 64.77 0)
+  (symbol (lib_id "Device:C") (at 184.15 64.77 0) (unit 1)
+    (in_bom yes) (on_board yes)
+    (property "Reference" "Cgps4" (id 0) (at 181.61 62.23 0)
+      (effects (font (size 1.27 1.27)) (justify left))
+    )
+    (property "Value" "100pF" (id 1) (at 184.15 67.31 0)
+      (effects (font (size 1.27 1.27)) (justify left))
+    )
+    (property "Footprint" "Capacitor_SMD:C_0603_1608Metric" (id 2) (at 185.1152 68.58 0)
+      (effects (font (size 1.27 1.27)) hide)
+    )
+    (property "Datasheet" "~" (id 3) (at 184.15 64.77 0)
+      (effects (font (size 1.27 1.27)) hide)
+    )
+    (pin "1")
+    (pin "2")
+  )
+  (symbol (lib_id "Device:C") (at 176.53 64.77 0) (unit 1)
+    (in_bom yes) (on_board yes)
+    (property "Reference" "Cgps3" (id 0) (at 173.99 62.23 0)
+      (effects (font (size 1.27 1.27)) (justify left))
+    )
+    (property "Value" "1uF" (id 1) (at 176.53 67.31 0)
+      (effects (font (size 1.27 1.27)) (justify left))
+    )
+    (property "Footprint" "Capacitor_SMD:C_0603_1608Metric" (id 2) (at 177.4952 68.58 0)
+      (effects (font (size 1.27 1.27)) hide)
+    )
+    (property "Datasheet" "~" (id 3) (at 176.53 64.77 0)
       (effects (font (size 1.27 1.27)) hide)
     )
@@
   )
   (symbol (lib_id "pspice:INDUCTOR") (at 161.29 60.96 0) (unit 1)
-    (in_bom yes) (on_board yes) (fields_autoplaced)
-    (property "Reference" "Lgps1" (id 0) (at 161.29 54.61 0))
-    (property "Value" "33nH" (id 1) (at 161.29 57.15 0))
+    (in_bom yes) (on_board yes)
+    (property "Reference" "Lgps1" (id 0) (at 161.29 55.88 0))
+    (property "Value" "33nH" (id 1) (at 161.29 58.42 0))
     (property "Footprint" "Inductor_SMD:L_0603_1608Metric" (id 2) (at 161.29 60.96 0)
       (effects (font (size 1.27 1.27)) hide)
@@
   (symbol (lib_id "Connector_Generic:Conn_01x05") (at 91.44 80.01 0) (unit 1)
     (in_bom yes) (on_board yes) (fields_autoplaced)
-    (property "Reference" "J1" (id 0) (at 93.98 78.7399 0)
-      (effects (font (size 1.27 1.27)) (justify left))
-    )
+    (property "Reference" "JCompass1" (id 0) (at 93.98 78.7399 0)
+      (effects (font (size 1.27 1.27)) (justify left))
+    )

Commit message: Aggiornamenti vari
Parts:
- JCompass1: value Conn_01x05 -> GY-271; footprint Connector_PinSocket_2.54mm:PinSocket_1x05_P2.54mm_Vertical -> mia_libreria:GY-271
