File: gps_compass_circuit_atmega328_7seg/gps_compass_atmega328.kicad_sch (KiCad schematic)
At the start: 7 parts, among them U3 ATmega328P-A, Y1 Crystal

Commit message: Aggiornamenti vari
Connections:
- net B6: now reaches U3.11 (PD7)
- no-connect marks 3 -> 2
