File: gps_compass_circuit_atmega328_7seg/gps_compass_display.kicad_sch (KiCad schematic)
At the start: 4 parts

Commit message: Aggiornato circuito
Parts:
- SWLed1: footprint Button_Switch_SMD:SW_SPST_Omron_B3FS-101xP -> Button_Switch_THT:SW_PUSH_6mm
Changed lines of the file:
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@@
       (effects (font (size 1.27 1.27)) hide)
     )
-    (property "Footprint" "Button_Switch_SMD:SW_SPST_Omron_B3FS-101xP" (id 2) (at 113.03 52.07 0)
+    (property "Footprint" "Button_Switch_THT:SW_PUSH_6mm" (id 2) (at 113.03 52.07 0)
       (effects (font (size 1.27 1.27)) hide)
     )

Commit message: upt circuit
Parts:
- JDisplay1: footprint (none) -> Connector_PinSocket_2.54mm:PinSocket_1x05_P2.54mm_Vertical
Changed lines of the file:
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@@
     (property "Reference" "JDisplay1" (id 0) (at 127 64.77 0))
     (property "Value" "Conn_01x05" (id 1) (at 127 67.31 0))
-    (property "Footprint" "" (id 2) (at 127 76.2 0)
+    (property "Footprint" "Connector_PinSocket_2.54mm:PinSocket_1x05_P2.54mm_Vertical" (id 2) (at 127 76.2 0)
       (effects (font (size 1.27 1.27)) hide)
     )

Commit message: Aggiornamenti vari
Parts:
- JDisplay1: footprint Connector_PinSocket_2.54mm:PinSocket_1x05_P2.54mm_Vertical -> mia_libreria:display_7_segm_4_digits
