File: gps_compass_circuit_atmega328_7seg/gps_compass_power.kicad_sch (KiCad schematic)
At the start: 11 parts, among them U4 MCP1700x-330xxTT

Commit message: Aggiornato circuito
Parts:
- removed C_sup2: 3.9v200F, Capacitor_THT:C_Rect_L9.0mm_W2.5mm_P7.50mm_MKT, symbol pspice:C
Other:
- moved on the sheet: C_sup1
Changed lines of the file:
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@@
   (junction (at 91.44 106.68) (diameter 0) (color 0 0 0 0)
   )
-  (junction (at 114.3 106.68) (diameter 0) (color 0 0 0 0)
+  (junction (at 110.49 106.68) (diameter 0) (color 0 0 0 0)
   )
   (junction (at 172.72 58.42) (diameter 0) (color 0 0 0 0)
@@
   (junction (at 130.81 60.96) (diameter 0) (color 0 0 0 0)
   )
-  (junction (at 100.33 106.68) (diameter 0) (color 0 0 0 0)
-  )
-  (junction (at 100.33 58.42) (diameter 0) (color 0 0 0 0)
-  )
-  (junction (at 114.3 58.42) (diameter 0) (color 0 0 0 0)
-  )
   (junction (at 91.44 58.42) (diameter 0) (color 0 0 0 0)
   )
   (junction (at 143.51 78.74) (diameter 0) (color 0 0 0 0)
   )
+  (junction (at 110.49 58.42) (diameter 0) (color 0 0 0 0)
+  )
   (wire (pts (xy 82.55 58.42) (xy 91.44 58.42))
     (stroke (width 0) (type default) (color 0 0 0 0))
@@
     (stroke (width 0) (type default) (color 0 0 0 0))
   )
-  (wire (pts (xy 114.3 58.42) (xy 116.84 58.42))
-    (stroke (width 0) (type default) (color 0 0 0 0))
-  )
   (wire (pts (xy 130.81 60.96) (xy 130.81 58.42))
     (stroke (width 0) (type default) (color 0 0 0 0))
@@
     (stroke (width 0) (type default) (color 0 0 0 0))
   )
-  (wire (pts (xy 114.3 106.68) (xy 143.51 106.68))
-    (stroke (width 0) (type default) (color 0 0 0 0))
-  )
   (wire (pts (xy 91.44 106.68) (xy 66.04 106.68))
     (stroke (width 0) (type default) (color 0 0 0 0))
   )
-  (wire (pts (xy 100.33 58.42) (xy 100.33 82.55))
+  (wire (pts (xy 110.49 58.42) (xy 110.49 82.55))
     (stroke (width 0) (type default) (color 0 0 0 0))
   )
@@
     (stroke (width 0) (type default) (color 0 0 0 0))
   )
-  (wire (pts (xy 114.3 95.25) (xy 114.3 106.68))
-    (stroke (width 0) (type default) (color 0 0 0 0))
-  )
-  (wire (pts (xy 100.33 58.42) (xy 114.3 58.42))
-    (stroke (width 0) (type default) (color 0 0 0 0))
-  )
   (wire (pts (xy 130.81 58.42) (xy 135.89 58.42))
     (stroke (width 0) (type default) (color 0 0 0 0))
@@
     (stroke (width 0) (type default) (color 0 0 0 0))
   )
-  (wire (pts (xy 91.44 106.68) (xy 100.33 106.68))
+  (wire (pts (xy 91.44 106.68) (xy 110.49 106.68))
+    (stroke (width 0) (type default) (color 0 0 0 0))
+  )
+  (wire (pts (xy 110.49 58.42) (xy 116.84 58.42))
     (stroke (width 0) (type default) (color 0 0 0 0))
   )
@@
     (stroke (width 0) (type default) (color 0 0 0 0))
   )
-  (wire (pts (xy 114.3 58.42) (xy 114.3 82.55))
-    (stroke (width 0) (type default) (color 0 0 0 0))
-  )
   (wire (pts (xy 189.23 87.63) (xy 200.66 87.63))
     (stroke (width 0) (type default) (color 0 0 0 0))
   )
-  (wire (pts (xy 100.33 106.68) (xy 114.3 106.68))
-    (stroke (width 0) (type default) (color 0 0 0 0))
-  )
-  (wire (pts (xy 100.33 95.25) (xy 100.33 106.68))
-    (stroke (width 0) (type default) (color 0 0 0 0))
-  )
-  (wire (pts (xy 91.44 58.42) (xy 100.33 58.42))
+  (wire (pts (xy 110.49 95.25) (xy 110.49 106.68))
+    (stroke (width 0) (type default) (color 0 0 0 0))
+  )
+  (wire (pts (xy 91.44 58.42) (xy 110.49 58.42))
     (stroke (width 0) (type default) (color 0 0 0 0))
   )
   (wire (pts (xy 66.04 106.68) (xy 66.04 114.3))
+    (stroke (width 0) (type default) (color 0 0 0 0))
+  )
+  (wire (pts (xy 110.49 106.68) (xy 143.51 106.68))
     (stroke (width 0) (type default) (color 0 0 0 0))
   )
@@
     (pin "2")
   )
-  (symbol (lib_id "pspice:C") (at 100.33 88.9 0) (unit 1)
+  (symbol (lib_id "pspice:C") (at 110.49 88.9 0) (unit 1)
     (in_bom yes) (on_board yes)
-    (property "Reference" "C_sup1" (id 0) (at 104.14 85.09 0)
-      (effects (font (size 1.27 1.27)) (justify left))
-    )
-    (property "Value" "3.9v200F" (id 1) (at 104.14 92.71 0)
-      (effects (font (size 1.27 1.27)) (justify left))
-    )
-    (property "Footprint" "Capacitor_THT:C_Rect_L9.0mm_W2.5mm_P7.50mm_MKT" (id 2) (at 100.33 88.9 0)
-      (effects (font (size 1.27 1.27)) hide)
-    )
-    (property "Datasheet" "~" (id 3) (at 100.33 88.9 0)
+    (property "Reference" "C_sup1" (id 0) (at 114.3 85.09 0)
+      (effects (font (size 1.27 1.27)) (justify left))
+    )
+    (property "Value" "3.9v200F" (id 1) (at 114.3 92.71 0)
+      (effects (font (size 1.27 1.27)) (justify left))
+    )
+    (property "Footprint" "Capacitor_THT:C_Rect_L9.0mm_W2.5mm_P7.50mm_MKT" (id 2) (at 110.49 88.9 0)
+      (effects (font (size 1.27 1.27)) hide)
+    )
+    (property "Datasheet" "~" (id 3) (at 110.49 88.9 0)
       (effects (font (size 1.27 1.27)) hide)
     )
@@
     (pin "6")
   )
-  (symbol (lib_id "pspice:C") (at 114.3 88.9 0) (unit 1)
-    (in_bom yes) (on_board yes)
-    (property "Reference" "C_sup2" (id 0) (at 118.11 85.09 0)
-      (effects (font (size 1.27 1.27)) (justify left))
-    )
-    (property "Value" "3.9v200F" (id 1) (at 118.11 92.71 0)
-      (effects (font (size 1.27 1.27)) (justify left))
-    )
-    (property "Footprint" "Capacitor_THT:C_Rect_L9.0mm_W2.5mm_P7.50mm_MKT" (id 2) (at 114.3 88.9 0)
-      (effects (font (size 1.27 1.27)) hide)
-    )
-    (property "Datasheet" "~https://www.digikey.it/it/products/detail/tecate-group/TPLC-3R8-200MR16X25/12417590" (id 3) (at 114.3 88.9 0)
-      (effects (font (size 1.27 1.27)) hide)
-    )
-    (pin "1")
-    (pin "2")
-  )
 )

Commit message: Aggiornamenti vari
Parts:
- SC_1, SC_2: footprint Connector_PinSocket_2.54mm:PinSocket_1x02_P2.54mm_Vertical -> mia_libreria:solar_panel
