File: gps_compass_circuit_atmega328_7seg/gps_compass.kicad_sch (KiCad schematic)
At the start: 0 parts

Commit message: Aggiornamenti vari
Parts:
- added C1: 0.1uF, Capacitor_SMD:C_0603_1608Metric, symbol Device:C
- added C2, C3: 22pF, Capacitor_SMD:C_0603_1608Metric, symbol Device:C
- added C_sup1: 3.9v200F, Capacitor_THT:C_Rect_L9.0mm_W2.5mm_P7.50mm_MKT, symbol pspice:C
- added Cdtr1: 0.1uF, Resistor_SMD:R_0603_1608Metric, symbol Device:C
- added Cgps1, Cgps2, Cgps4: 100pF, Capacitor_SMD:C_0603_1608Metric, symbol Device:C
- added Cgps3: 1uF, Capacitor_SMD:C_0603_1608Metric, symbol Device:C
- added Cv1: 1uF, Capacitor_SMD:C_0603_1608Metric, symbol pspice:C
- added D1: MBR0530, Diode_SMD:D_SOD-123, symbol Diode:MBR0530
- added D2: BZV55B3V9, Diode_THT:D_A-405_P7.62mm_Horizontal, symbol Diode:BZV55B3V9
- added JCompass1: GY-271, mia_libreria:GY-271, symbol Connector_Generic:Conn_01x05
- added JDisplay1: Conn_01x05, mia_libreria:display_7_segm_4_digits, symbol Connector_Generic:Conn_01x05
- added JGPS1: Conn_01x05, Connector_PinSocket_2.54mm:PinSocket_1x05_P2.54mm_Vertical, symbol Connector_Generic:Conn_01x05
- added JMicroSD1: Micro_SD_Card, Connector_Card:microSD_HC_Molex_47219-2001, symbol Connector:Micro_SD_Card
- added JPFTDI1: FTDI_basic, Connector_PinSocket_2.54mm:PinSocket_1x06_P2.54mm_Horizontal, symbol Connector_Generic:Conn_01x06
- added Led1: LED, LED_THT:LED_D3.0mm, symbol Device:LED
- added Lgps1, Lgps2: 33nH, Inductor_SMD:L_0603_1608Metric, symbol pspice:INDUCTOR
- added R1: 1M, Capacitor_SMD:C_0603_1608Metric, symbol pspice:R
- added R2: 100K, Capacitor_SMD:C_0603_1608Metric, symbol pspice:R
- added R_cells1: R59, Resistor_SMD:R_0603_1608Metric, symbol Device:R
- added Rgps1, Rgps2: 200R, Resistor_SMD:R_0603_1608Metric, symbol pspice:R
- added Rled1: 700R, Resistor_SMD:R_0603_1608Metric, symbol pspice:R
- added Rreset1: 10k, Resistor_SMD:R_0603_1608Metric, symbol Device:R
- added Rscl1, Rsda1: 10K, Resistor_SMD:R_0603_1608Metric, symbol Device:R
- added SC_1, SC_2: Solar_Cell, mia_libreria:solar_panel, symbol Device:Solar_Cell
- added SW1, SW2, SW3, SW4, SW5, SW6: SW_SPST, Button_Switch_THT:SW_PUSH_6mm, symbol Switch:SW_SPST
- added SWLed1, SWReset1: SW_Reset, Button_Switch_THT:SW_PUSH_6mm, symbol Switch:SW_DIP_x01
- added SW_MCU1, SW_main_switch1: SW_DPDT_x2, Connector_PinSocket_2.54mm:PinSocket_1x03_P2.54mm_Vertical, symbol Switch:SW_DPDT_x2
- added U3: ATmega328P-A, Package_QFP:TQFP-32_7x7mm_P0.8mm, symbol MCU_Microchip_ATmega:ATmega328P-A
- added U4: MCP1700x-330xxTT, Package_TO_SOT_SMD:SOT-23, symbol Regulator_Linear:MCP1700x-330xxTT
- added Y1: Crystal, Crystal:Resonator-2Pin_W10.0mm_H5.0mm, symbol Device:Crystal
Connections:
- new net: Led1.1 (K), SWLed1.2
- new net: Led1.2 (A), Rled1.1
- new net: JGPS1.1 (Pin_1), Rgps1.2
- new net: JGPS1.2 (Pin_2), Rgps2.2
- new net: Cgps3.1, Cgps4.1, JGPS1.3 (Pin_3), Lgps1.2
- new net: Cgps3.2, Cgps4.2, JGPS1.4 (Pin_4), Lgps2.2
- new net: Cdtr1.2, JPFTDI1.1 (Pin_1)
- new net: C_sup1.1, D1.1 (K), D2.1 (K), SW_main_switch1.2 (B)
- new net: D1.2 (A), R_cells1.1
- new net: C2.1, U3.7 (XTAL1/PB6), Y1.2
- new net: C1.2, U3.20 (AREF)
- new net: R1.2, R2.1, U3.22 (ADC7)
- new net: C3.1, U3.8 (XTAL2/PB7), Y1.1
- new net: R_cells1.2, SC_1.1 (+)
- new net: SC_1.2 (-), SC_2.1 (+)
- new net +3V3: JCompass1.1 (Pin_1), JDisplay1.2 (Pin_2), JMicroSD1.4 (VDD), JPFTDI1.4 (Pin_4), Rled1.2, Rreset1.1, Rscl1.1, Rsda1.1, SW_MCU1.3 (C), U3.18 (AVCC), U3.4 (VCC), U3.6 (VCC)
- new net B1: SW1.2 (B), U3.12 (PB0)
- new net B2: SW2.2 (B), U3.13 (PB1)
- new net B3: SW3.2 (B), U3.24 (PC1)
- new net B4: SW4.2 (B), U3.25 (PC2)
- new net B5: SW5.2 (B), U3.26 (PC3)
- new net B6: SW6.2 (B), U3.11 (PD7)
- new net Display_CS: JDisplay1.5 (Pin_5), U3.10 (PD6)
- new net Display_DA: JDisplay1.3 (Pin_3), U3.2 (PD4)
- new net Display_WR: JDisplay1.4 (Pin_4), U3.9 (PD5)
- new net FTDI_RX: JPFTDI1.3 (Pin_3), U3.30 (PD0)
- new net FTDI_TX: JPFTDI1.2 (Pin_2), U3.31 (PD1)
- new net GND: C1.1, C2.2, C3.2, C_sup1.2, Cgps1.2, Cgps2.2, Cv1.2, D2.2 (A), JCompass1.2 (Pin_2), JDisplay1.1 (Pin_1), JMicroSD1.3 (CMD), JMicroSD1.6 (VSS), JMicroSD1.9 (SHIELD), JPFTDI1.5 (Pin_5), JPFTDI1.6 (Pin_6), Lgps2.1, R2.2, SC_2.2 (-), SW1.1 (A), SW2.1 (A), SW3.1 (A), SW4.1 (A), SW5.1 (A), SW6.1 (A), SWLed1.1, SWReset1.1, U3.21 (GND), U3.3 (GND), U3.5 (GND), U4.1 (GND)
- new net Power_level: R1.1, SW_main_switch1.3 (C), U4.3 (VI)
- new net RESET: Cdtr1.1, Rreset1.2, SWReset1.2, U3.29 (~{RESET}/PC6)
- new net SCL: JCompass1.3 (Pin_3), Rscl1.2, U3.28 (PC5)
- new net SDA: JCompass1.4 (Pin_4), Rsda1.2, U3.27 (PC4)
- new net VCC: Cv1.1, Lgps1.1, SW_MCU1.2 (B), U4.2 (VO)
- new net gps_rx: Cgps2.1, Rgps2.1, U3.1 (PD3)
- new net gps_tx: Cgps1.1, Rgps1.1, U3.32 (PD2)
- new net microSD_cs: JMicroSD1.1 (DAT2), U3.14 (PB2)
- new net microSD_di: JMicroSD1.2 (DAT3/CD), U3.15 (PB3)
- new net microSD_do: JMicroSD1.7 (DAT0), U3.17 (PB5)
- new net microSD_sclk: JMicroSD1.5 (CLK), U3.16 (PB4)
- no-connect marks 0 -> 5
Other:
- removed sheet ATMEGA328
- removed sheet Display
- removed sheet GPSeCompass
- removed sheet Periferiche
- removed sheet power
