File: gps_compass_circuit_esp32_battery/gps_compass.kicad_sch (KiCad schematic)
At the start: 39 parts, among them J1 USB_C_Receptacle_PowerOnly_6P, Q1 MMBTA92, U1 MCP1700x-330xxTT, U3 LTC4054ES5-4.2

Commit message: Aggiornamenti vari
Parts:
- removed GY-271: Conn_01x05_Shielded, mia_libreria:GY-271, symbol Connector_Generic_Shielded:Conn_01x05_Shielded
- removed L1: 120R@100Mhz, Inductor_SMD:L_0805_2012Metric_Pad1.15x1.40mm_HandSolder, symbol Device:L
- removed Oled1: display_oled, mia_libreria:Display_i2c_128x64, symbol Connector_Generic_Shielded:Conn_01x04_Shielded
- removed Serial1: Conn_01x03_Shielded, Connector_PinSocket_2.54mm:PinSocket_1x03_P2.54mm_Vertical, symbol Connector_Generic_Shielded:Conn_01x03_Shielded
- removed lcd1: display_lcd, mia_libreria:display_7_segm_4_digits, symbol Connector_Generic_Shielded:Conn_01x05_Shielded
- added GY-271: Conn_01x05_Socket, mia_libreria:GY-271, symbol Connector:Conn_01x05_Socket
- added LCD1: Conn_01x05_Socket, mia_libreria:display_7_segm_4_digits, symbol Connector:Conn_01x05_Socket
- added Oled1: Conn_01x04_Socket, mia_libreria:Display_i2c_128x64, symbol Connector:Conn_01x04_Socket
- added Serial1: Conn_01x03_Socket, Connector_PinSocket_2.54mm:PinSocket_1x03_P2.54mm_Vertical, symbol Connector:Conn_01x03_Socket
Connections:
- net +3V3: now also ESP32.2 (B), MAIN1.1 (A)
- net GND: now also GY-271.2 (Pin_2), LCD1.1 (Pin_1), Oled1.1 (Pin_1), Serial1.3 (Pin_3)
- net SCL: now also GY-271.3 (Pin_3), Oled1.3 (Pin_3)
- net SDA: now also GY-271.4 (Pin_4), Oled1.4 (Pin_4)
- net VCC: now also GY-271.1 (Pin_1), LCD1.2 (Pin_2), Oled1.2 (Pin_2)
- net lcd_cs: now also LCD1.5 (Pin_5)
- net lcd_data: now also LCD1.3 (Pin_3)
- net lcd_wr: now also LCD1.4 (Pin_4)
- net at ESP32-S1.34 (RXD0/IO3): now also Serial1.2 (Pin_2)
- net at ESP32-S1.35 (TXD0/IO1): now also Serial1.1 (Pin_1)
- no-connect marks 24 -> 21

Commit message: Aggiornamenti vari
Parts:
- removed ESP32: SW_SPDT, Button_Switch_SMD:SW_SPDT_PCM12, symbol Switch:SW_SPDT
- added ESP1: SW_SPDT, Button_Switch_SMD:SW_SPDT_PCM12, symbol Switch:SW_SPDT
- added R10: 100K, Resistor_SMD:R_0603_1608Metric_Pad0.98x0.95mm_HandSolder, symbol Device:R
- added R9: 27K, Resistor_SMD:R_0603_1608Metric_Pad0.98x0.95mm_HandSolder, symbol Device:R
Connections:
- net +3V3: now also C6.1, C7.1, U1.2 (VO), ESP1.2 (B); no longer MAIN1.1 (A)
- net GND: now also R10.2
- net SCL: now also GPS1.12 (SCL)
- net SDA: now also GPS1.9 (SDA)
- net VCC: now also ESP1.1 (A)
- net at BT1.1 (+), C1.1, Q1.3 (C)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: now also MAIN1.2 (B); no longer C5.1, U1.3 (VI)
- net battery_level: now reaches ESP32-S1.9 (IO33)
- net battery_level: now also R10.1, R9.2
- new net +BATT: C5.1, MAIN1.1 (A), R9.1, U1.3 (VI)
- no-connect marks 21 -> 18
Other:
- moved on the sheet: C3, C4
